File: electric-imp-version.sch (EAGLE design)
At the start: 44 parts, among them Q1 DMG2307L-7, U1 ELECTRIC_IMP, U2 TPS62172, U3 ATSHA204-TSU, U4 MCP73831, U5 CD74HC4067-SSOPCD74HC4067, U6 CD74HC4067-SSOPCD74HC4067, U7 LTC6904LTC6904, X1 USBSMD

Commit message: Cleaning up traces
Parts:
- removed JP9: FIDUCIALUFIDUCIAL, SparkFun:FIDUCIALUFIDUCIAL
- C4: device SparkFun-Passives:CAP0402-CAP -> SparkFun-Capacitors:CAP0603-CAP
- R4: value 330k -> 330
- renumbered C13 to C7
Other:
- moved on the sheet: C8, R7
Changed lines of the file:
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@@
 <part name="P+4" library="SparkFun-Aesthetics" deviceset="3.3V" device=""/>
 <part name="GND6" library="SparkFun-Aesthetics" deviceset="GND" device=""/>
-<part name="C4" library="SparkFun-Passives" deviceset="CAP" device="0402-CAP" value="0.1uF"/>
 <part name="C2" library="SparkFun-Passives" deviceset="CAP" device="0805" value="22uF"/>
 <part name="L1" library="SparkFun-Passives" deviceset="INDUCTOR" device="VLF4012A" value="2.2uH"/>
@@
 <part name="U$5" library="SparkFun-Aesthetics" deviceset="OSHW-LOGO" device="S"/>
 <part name="JP8" library="SparkFun" deviceset="FIDUCIAL" device="UFIDUCIAL"/>
-<part name="JP9" library="SparkFun" deviceset="FIDUCIAL" device="UFIDUCIAL"/>
 <part name="S1" library="RHD2000" deviceset="OMNETICS_A79025" device=""/>
 <part name="U$3" library="autoimpedance" deviceset="AD5933" device=""/>
@@
 <part name="C3" library="SparkFun-Passives" deviceset="CAP" device="1210" value="4.7uF"/>
 <part name="GND12" library="SparkFun-Aesthetics" deviceset="GND" device=""/>
-<part name="R4" library="SparkFun-Passives" deviceset="RESISTOR" device="0402-RES" value="330k"/>
+<part name="R4" library="SparkFun-Passives" deviceset="RESISTOR" device="0402-RES" value="330"/>
 <part name="D1" library="SparkFun-LED" deviceset="LED-GREEN" device="0603" value="GREEN"/>
 <part name="R5" library="SparkFun-Passives" deviceset="RESISTOR" device="0402-RES" value="2k"/>
@@
 <part name="GND26" library="SparkFun-Aesthetics" deviceset="GND" device=""/>
 <part name="P+19" library="SparkFun-Aesthetics" deviceset="3.3V" device=""/>
-<part name="C13" library="SparkFun-Capacitors" deviceset="CAP" device="0603-CAP" value="0.1uF"/>
+<part name="C7" library="SparkFun-Capacitors" deviceset="CAP" device="0603-CAP" value="0.1uF"/>
 <part name="GND28" library="SparkFun-Aesthetics" deviceset="GND" device=""/>
 <part name="P+21" library="SparkFun-Aesthetics" deviceset="3.3V" device=""/>
@@
 <part name="GND19" library="SparkFun-Aesthetics" deviceset="GND" device=""/>
 <part name="P+14" library="SparkFun-Aesthetics" deviceset="3.3V" device=""/>
+<part name="C4" library="SparkFun-Capacitors" deviceset="CAP" device="0603-CAP" value="0.1uF"/>
 </parts>
 <sheets>
@@
 <instance part="P+4" gate="G$1" x="22.86" y="45.72" rot="MR0"/>
 <instance part="GND6" gate="1" x="22.86" y="17.78" rot="MR0"/>
-<instance part="C4" gate="G$1" x="15.24" y="27.94" rot="MR0"/>
 <instance part="C2" gate="G$1" x="124.46" y="144.78"/>
 <instance part="L1" gate="G$1" x="109.22" y="152.4" smashed="yes" rot="R90">
@@
 <instance part="U$5" gate="G$1" x="132.08" y="10.16"/>
 <instance part="JP8" gate="G$1" x="243.84" y="33.02"/>
-<instance part="JP9" gate="G$1" x="243.84" y="27.94"/>
 <instance part="S1" gate="A" x="121.92" y="106.68" rot="R270"/>
 <instance part="U$3" gate="G$1" x="167.64" y="157.48"/>
@@
 <instance part="U$6" gate="G$1" x="213.36" y="127"/>
 <instance part="R6" gate="G$1" x="91.44" y="45.72" rot="MR90"/>
-<instance part="R7" gate="G$1" x="96.52" y="43.18" rot="MR90"/>
+<instance part="R7" gate="G$1" x="101.6" y="43.18" rot="MR90"/>
 <instance part="P+6" gate="G$1" x="91.44" y="50.8" rot="MR0"/>
-<instance part="P+7" gate="G$1" x="96.52" y="48.26" rot="MR0"/>
+<instance part="P+7" gate="G$1" x="101.6" y="48.26" rot="MR0"/>
 <instance part="P+8" gate="G$1" x="187.96" y="144.78" rot="R180"/>
 <instance part="GND15" gate="1" x="193.04" y="152.4"/>
@@
 <instance part="GND8" gate="1" x="152.4" y="53.34" rot="MR0"/>
 <instance part="GND20" gate="1" x="182.88" y="68.58" rot="MR270"/>
-<instance part="C8" gate="G$1" x="137.16" y="63.5"/>
-<instance part="GND23" gate="1" x="137.16" y="58.42"/>
-<instance part="P+16" gate="G$1" x="137.16" y="68.58"/>
+<instance part="C8" gate="G$1" x="132.08" y="63.5"/>
+<instance part="GND23" gate="1" x="132.08" y="55.88"/>
+<instance part="P+16" gate="G$1" x="132.08" y="71.12"/>
 <instance part="U7" gate="G$1" x="200.66" y="106.68"/>
 <instance part="U8" gate="G$1" x="162.56" y="68.58"/>
@@
 <instance part="GND26" gate="1" x="172.72" y="101.6"/>
 <instance part="P+19" gate="G$1" x="172.72" y="116.84"/>
-<instance part="C13" gate="G$1" x="226.06" y="106.68"/>
+<instance part="C7" gate="G$1" x="226.06" y="106.68"/>
 <instance part="GND28" gate="1" x="226.06" y="101.6"/>
 <instance part="P+21" gate="G$1" x="226.06" y="111.76"/>
@@
 <instance part="GND19" gate="1" x="180.34" y="124.46"/>
 <instance part="P+14" gate="G$1" x="139.7" y="99.06" rot="R180"/>
+<instance part="C4" gate="G$1" x="15.24" y="27.94"/>
 </instances>
 <busses>
@@
 <wire x1="27.94" y1="27.94" x2="22.86" y2="27.94" width="0.1524" layer="91"/>
 <wire x1="22.86" y1="27.94" x2="22.86" y2="22.86" width="0.1524" layer="91"/>
-<pinref part="C4" gate="G$1" pin="2"/>
 <wire x1="22.86" y1="22.86" x2="22.86" y2="20.32" width="0.1524" layer="91"/>
 <wire x1="15.24" y1="25.4" x2="15.24" y2="22.86" width="0.1524" layer="91"/>
 <wire x1="15.24" y1="22.86" x2="22.86" y2="22.86" width="0.1524" layer="91"/>
 <junction x="22.86" y="22.86"/>
+<pinref part="C4" gate="G$1" pin="2"/>
 </segment>
 <segment>
@@
 <pinref part="C8" gate="G$1" pin="2"/>
 <pinref part="GND23" gate="1" pin="GND"/>
+<wire x1="132.08" y1="60.96" x2="132.08" y2="58.42" width="0.1524" layer="91"/>
 </segment>
 <segment>
@@
 </segment>
 <segment>
-<pinref part="C13" gate="G$1" pin="2"/>
+<pinref part="C7" gate="G$1" pin="2"/>
 <pinref part="GND28" gate="1" pin="GND"/>
 </segment>
@@
 <wire x1="27.94" y1="33.02" x2="22.86" y2="33.02" width="0.1524" layer="91"/>
 <wire x1="22.86" y1="33.02" x2="22.86" y2="38.1" width="0.1524" layer="91"/>
-<pinref part="C4" gate="G$1" pin="1"/>
 <wire x1="22.86" y1="38.1" x2="22.86" y2="45.72" width="0.1524" layer="91"/>
 <wire x1="15.24" y1="33.02" x2="15.24" y2="38.1" width="0.1524" layer="91"/>
 <wire x1="15.24" y1="38.1" x2="22.86" y2="38.1" width="0.1524" layer="91"/>
 <junction x="22.86" y="38.1"/>
+<pinref part="C4" gate="G$1" pin="1"/>
 </segment>
 <segment>
@@
 <pinref part="C8" gate="G$1" pin="1"/>
 <pinref part="P+16" gate="G$1" pin="3.3V"/>
+<wire x1="132.08" y1="68.58" x2="132.08" y2="71.12" width="0.1524" layer="91"/>
 </segment>
 <segment>
@@
 </segment>
 <segment>
-<pinref part="C13" gate="G$1" pin="1"/>
+<pinref part="C7" gate="G$1" pin="1"/>
 <pinref part="P+21" gate="G$1" pin="3.3V"/>
 <pinref part="U7" gate="G$1" pin="OE"/>
@@
 <pinref part="U1" gate="G$1" pin="2(CMD)"/>
 <label x="83.82" y="38.1" size="1.778" layer="95"/>
-<wire x1="83.82" y1="38.1" x2="96.52" y2="38.1" width="0.1524" layer="91"/>
+<wire x1="83.82" y1="38.1" x2="101.6" y2="38.1" width="0.1524" layer="91"/>
 <pinref part="R7" gate="G$1" pin="1"/>
 </segment>

Commit message: Fix layout
Parts:
- removed FRAME1: FRAME-LETTER, SparkFun-Aesthetics:FRAME-LETTER
Changed lines of the file:
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@@
 </classes>
 <parts>
-<part name="FRAME1" library="SparkFun-Aesthetics" deviceset="FRAME-LETTER" device=""/>
 <part name="U1" library="SparkFun-RF" deviceset="ELECTRIC_IMP" device=""/>
 <part name="P+2" library="SparkFun-Aesthetics" deviceset="3.3V" device=""/>
@@
 </plain>
 <instances>
-<instance part="FRAME1" gate="G$1" x="0" y="0"/>
-<instance part="FRAME1" gate="G$2" x="147.32" y="0"/>
 <instance part="U1" gate="G$1" x="71.12" y="30.48" rot="MR0"/>
 <instance part="P+2" gate="G$1" x="55.88" y="45.72" rot="MR0"/>

Commit message: Aesthetic fixes
Parts:
- added FRAME1: FRAME-LETTER, SparkFun-Aesthetics:FRAME-LETTER
- renumbered JP3 to JP1, S1 to OMNETICS, U$3 to IC1, U$4 to IC3, U$6 to IC2, U$8 to MUX3X2, U1 to SD, U2 to CONV, U3 to ID, U4 to CHARGE, U5 to MUX16A, U6 to MUX16B, U7 to CLK, U8 to SR, X1 to USB

Commit message: Fix LM234 channel mapping
Parts:
- removed IC2: LM234, josh:LM234
- added U$2: LM234, josh:LM234
Connections:
- net CURRENT_SOURCE: now also U$2.V–; no longer IC2.V-2
- net LM234EN: now also U$2.V+; no longer IC2.V+
- net W: now also U$2.ADJ; no longer IC2.R
Changed lines of the file:
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@@
 <part name="GND13" library="SparkFun-Aesthetics" deviceset="GND" device=""/>
 <part name="GND14" library="SparkFun-Aesthetics" deviceset="GND" device=""/>
-<part name="IC2" library="josh" deviceset="LM234" device=""/>
 <part name="R6" library="SparkFun-Passives" deviceset="RESISTOR" device="0402-RES" value="4.7k"/>
 <part name="R7" library="SparkFun-Passives" deviceset="RESISTOR" device="0402-RES" value="4.7k"/>
@@
 <part name="C4" library="SparkFun-Capacitors" deviceset="CAP" device="0603-CAP" value="0.1uF"/>
 <part name="FRAME1" library="SparkFun-Aesthetics" deviceset="FRAME-LETTER" device=""/>
+<part name="U$2" library="josh" deviceset="LM234" device=""/>
 </parts>
 <sheets>
@@
 <instance part="GND13" gate="1" x="71.12" y="162.56"/>
 <instance part="GND14" gate="1" x="76.2" y="160.02"/>
-<instance part="IC2" gate="G$1" x="213.36" y="127"/>
 <instance part="R6" gate="G$1" x="91.44" y="45.72" rot="MR90"/>
 <instance part="R7" gate="G$1" x="101.6" y="43.18" rot="MR90"/>
@@
 <instance part="FRAME1" gate="G$1" x="0" y="0"/>
 <instance part="FRAME1" gate="G$2" x="147.32" y="0"/>
+<instance part="U$2" gate="G$1" x="215.9" y="116.84"/>
 </instances>
 <busses>
@@
 <net name="LM234EN" class="0">
 <segment>
-<pinref part="IC2" gate="G$1" pin="V+"/>
-<wire x1="213.36" y1="144.78" x2="205.74" y2="144.78" width="0.1524" layer="91"/>
-<label x="203.2" y="144.78" size="1.778" layer="95"/>
+<wire x1="215.9" y1="134.62" x2="205.74" y2="134.62" width="0.1524" layer="91"/>
+<label x="200.66" y="134.62" size="1.778" layer="95"/>
+<pinref part="U$2" gate="G$1" pin="V+"/>
 </segment>
 <segment>
@@
 </segment>
 <segment>
-<pinref part="IC2" gate="G$1" pin="R"/>
-<wire x1="213.36" y1="142.24" x2="205.74" y2="142.24" width="0.1524" layer="91"/>
-<label x="205.74" y="142.24" size="1.778" layer="95"/>
+<wire x1="215.9" y1="132.08" x2="203.2" y2="132.08" width="0.1524" layer="91"/>
+<label x="205.74" y="132.08" size="1.778" layer="95"/>
+<pinref part="U$2" gate="G$1" pin="ADJ"/>
 </segment>
 </net>
@@
 </segment>
 <segment>
-<pinref part="IC2" gate="G$1" pin="V-2"/>
-<wire x1="213.36" y1="137.16" x2="205.74" y2="137.16" width="0.1524" layer="91"/>
-<label x="205.74" y="137.16" size="1.778" layer="95"/>
-</segment>
-<segment>
+<wire x1="215.9" y1="129.54" x2="195.58" y2="129.54" width="0.1524" layer="91"/>
+<label x="195.58" y="127" size="1.778" layer="95"/>
+<pinref part="U$2" gate="G$1" pin="V–"/>
+</segment>
+<segment>

Commit message: Update BOM
Parts:
- renumbered U$2 to IC2
Changed lines of the file:
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@@
 <part name="C4" library="SparkFun-Capacitors" deviceset="CAP" device="0603-CAP" value="0.1uF"/>
 <part name="FRAME1" library="SparkFun-Aesthetics" deviceset="FRAME-LETTER" device=""/>
-<part name="U$2" library="josh" deviceset="LM234" device=""/>
+<part name="IC2" library="josh" deviceset="LM234" device=""/>
 </parts>
 <sheets>
@@
 <instance part="FRAME1" gate="G$1" x="0" y="0"/>
 <instance part="FRAME1" gate="G$2" x="147.32" y="0"/>
-<instance part="U$2" gate="G$1" x="215.9" y="116.84"/>
+<instance part="IC2" gate="G$1" x="215.9" y="116.84"/>
 </instances>
 <busses>
@@
 <wire x1="215.9" y1="134.62" x2="205.74" y2="134.62" width="0.1524" layer="91"/>
 <label x="200.66" y="134.62" size="1.778" layer="95"/>
-<pinref part="U$2" gate="G$1" pin="V+"/>
+<pinref part="IC2" gate="G$1" pin="V+"/>
 </segment>
 <segment>
@@
 <wire x1="215.9" y1="132.08" x2="203.2" y2="132.08" width="0.1524" layer="91"/>
 <label x="205.74" y="132.08" size="1.778" layer="95"/>
-<pinref part="U$2" gate="G$1" pin="ADJ"/>
+<pinref part="IC2" gate="G$1" pin="ADJ"/>
 </segment>
 </net>
@@
 <wire x1="215.9" y1="129.54" x2="195.58" y2="129.54" width="0.1524" layer="91"/>
 <label x="195.58" y="127" size="1.778" layer="95"/>
-<pinref part="U$2" gate="G$1" pin="V–"/>
-</segment>
-<segment>
+<pinref part="IC2" gate="G$1" pin="V–"/>
+</segment>
+<segment>
